File: kicad/Raspberry pico board.kicad_pcb (KiCad board)
At the start: 2 copper layers, 24.8 x 96.5 mm, 11 parts, among them J1 Conn_01x20_Socket, J2 Conn_01x20_Socket, U2 MCP3301, U3 OPA340P, U4 C12666MA, U5 SN74AHCT125N, U6 SN74AHCT125N, U7 MCP1541-I/TO

Commit message: Schematic V2.0 finally made it work :)
Parts:
- moved U2 0.18 mm to (137.9, 87.1)
Changed lines of the file:
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@@
 	(footprint "Library JII FP:MCP3301_BI_P"
 		(layer "F.Cu")
-		(at 137.795 86.995)
+		(at 137.922 87.122)
 		(tags "MCP3301-BI/P ")
 		(property "Reference" "U2"
@@
 	)
 	(segment
-		(start 147.955 80.645)
-		(end 148.59 80.01)
-		(width 0.2)
-		(layer "F.Cu")
-		(net "Net-(U2-Vref)")
-	)
-	(segment
-		(start 142.24 86.995)
-		(end 145.415 83.82)
-		(width 0.2)
-		(layer "F.Cu")
-		(net "Net-(U2-Vref)")
-	)
-	(segment
-		(start 147.955 82.55)
-		(end 147.955 80.645)
-		(width 0.2)
-		(layer "F.Cu")
-		(net "Net-(U2-Vref)")
-	)
-	(segment
-		(start 137.795 86.995)
-		(end 142.24 86.995)
-		(width 0.2)
-		(layer "F.Cu")
-		(net "Net-(U2-Vref)")
-	)
-	(segment
-		(start 146.685 83.82)
-		(end 147.955 82.55)
-		(width 0.2)
-		(layer "F.Cu")
-		(net "Net-(U2-Vref)")
-	)
-	(segment
-		(start 145.415 83.82)
-		(end 146.685 83.82)
-		(width 0.2)
-		(layer "F.Cu")
-		(net "Net-(U2-Vref)")
-	)
-	(segment
-		(start 148.59 80.01)
-		(end 150.495 80.01)
-		(width 0.2)
-		(layer "F.Cu")
-		(net "Net-(U2-Vref)")
-	)
-	(segment
-		(start 136.525 105.41)
-		(end 135.255 104.14)
-		(width 0.2)
-		(layer "F.Cu")
-		(net "Net-(U2-CLK)")
-	)
-	(segment
-		(start 137.795 105.41)
-		(end 136.525 105.41)
-		(width 0.2)
-		(layer "F.Cu")
-		(net "Net-(U2-CLK)")
-	)
-	(segment
-		(start 135.255 104.14)
-		(end 135.255 98.425)
-		(width 0.2)
-		(layer "F.Cu")
-		(net "Net-(U2-CLK)")
-	)
-	(segment
-		(start 135.255 98.425)
-		(end 136.525 98.425)
-		(width 0.2)
-		(layer "F.Cu")
-		(net "Net-(U2-CLK)")
-	)
-	(segment
-		(start 136.525 98.425)
-		(end 145.415 89.535)
-		(width 0.2)
-		(layer "F.Cu")
-		(net "Net-(U2-CLK)")
-	)
-	(segment
-		(start 132.715 86.995)
-		(end 132.715 90.19)
-		(width 0.2)
-		(layer "B.Cu")
-		(net "Net-(U2-IN+)")
-	)
-	(segment
-		(start 135.255 89.535)
-		(end 137.795 89.535)
-		(width 0.2)
-		(layer "B.Cu")
-		(net "Net-(U2-IN+)")
-	)
-	(segment
-		(start 132.715 90.19)
-		(end 134.6 90.19)
-		(width 0.2)
-		(layer "B.Cu")
-		(net "Net-(U2-IN+)")
-	)
-	(segment
-		(start 134.6 90.19)
-		(end 135.255 89.535)
-		(width 0.2)
-		(layer "B.Cu")
-		(net "Net-(U2-IN+)")
-	)
-	(segment
-		(start 142.24 108.585)
-		(end 142.24 96.52)
-		(width 0.2)
-		(layer "F.Cu")
-		(net "Net-(U2-~{CS}{slash}SHDN)")
-	)
-	(segment
-		(start 137.795 113.03)
-		(end 142.24 108.585)
-		(width 0.2)
-		(layer "F.Cu")
-		(net "Net-(U2-~{CS}{slash}SHDN)")
-	)
-	(segment
-		(start 142.24 96.52)
-		(end 144.145 94.615)
-		(width 0.2)
-		(layer "F.Cu")
-		(net "Net-(U2-~{CS}{slash}SHDN)")
-	)
-	(segment
-		(start 144.145 94.615)
-		(end 145.415 94.615)
-		(width 0.2)
-		(layer "F.Cu")
-		(net "Net-(U2-~{CS}{slash}SHDN)")
-	)
-	(segment
 		(start 139.065 78.74)
 		(end 137.795 78.74)
@@
 	)
 	(segment
+		(start 132.715 86.995)
+		(end 132.715 90.19)
+		(width 0.2)
+		(layer "B.Cu")
+		(net "Net-(U2-IN+)")
+	)
+	(segment
+		(start 135.255 89.535)
+		(end 137.795 89.535)
+		(width 0.2)
+		(layer "B.Cu")
+		(net "Net-(U2-IN+)")
+	)
+	(segment
+		(start 132.715 90.19)
+		(end 134.6 90.19)
+		(width 0.2)
+		(layer "B.Cu")
+		(net "Net-(U2-IN+)")
+	)
+	(segment
+		(start 134.6 90.19)
+		(end 135.255 89.535)
+		(width 0.2)
+		(layer "B.Cu")
+		(net "Net-(U2-IN+)")
+	)
+	(segment
+		(start 130.175 95.25)
+		(end 137.795 102.87)
+		(width 0.2)
+		(layer "B.Cu")
+		(net "Net-(J2-Pin_17)")
+	)
+	(segment
+		(start 133.35 67.31)
+		(end 130.175 70.485)
+		(width 0.2)
+		(layer "B.Cu")
+		(net "Net-(J2-Pin_17)")
+	)
+	(segment
+		(start 130.175 70.485)
+		(end 130.175 95.25)
+		(width 0.2)
+		(layer "B.Cu")
+		(net "Net-(J2-Pin_17)")
+	)
+	(segment
+		(start 136.525 105.41)
+		(end 135.255 104.14)
+		(width 0.2)
+		(layer "F.Cu")
+		(net "Net-(U2-CLK)")
+	)
+	(segment
+		(start 137.795 105.41)
+		(end 136.525 105.41)
+		(width 0.2)
+		(layer "F.Cu")
+		(net "Net-(U2-CLK)")
+	)
+	(segment
+		(start 135.255 104.14)
+		(end 135.255 98.425)
+		(width 0.2)
+		(layer "F.Cu")
+		(net "Net-(U2-CLK)")
+	)
+	(segment
+		(start 135.255 98.425)
+		(end 136.525 98.425)
+		(width 0.2)
+		(layer "F.Cu")
+		(net "Net-(U2-CLK)")
+	)
+	(segment
+		(start 136.525 98.425)
+		(end 145.415 89.535)
+		(width 0.2)
+		(layer "F.Cu")
+		(net "Net-(U2-CLK)")
+	)
+	(segment
 		(start 134.855 104.305685)
 		(end 134.855 98.259315)
@@
 	)
 	(segment
+		(start 142.24 108.585)
+		(end 142.24 96.52)
+		(width 0.2)
+		(layer "F.Cu")
+		(net "Net-(U2-~{CS}{slash}SHDN)")
+	)
+	(segment
+		(start 137.795 113.03)
+		(end 142.24 108.585)
+		(width 0.2)
+		(layer "F.Cu")
+		(net "Net-(U2-~{CS}{slash}SHDN)")
+	)
+	(segment
+		(start 142.24 96.52)
+		(end 144.145 94.615)
+		(width 0.2)
+		(layer "F.Cu")
+		(net "Net-(U2-~{CS}{slash}SHDN)")
+	)
+	(segment
+		(start 144.145 94.615)
+		(end 145.415 94.615)
+		(width 0.2)
+		(layer "F.Cu")
+		(net "Net-(U2-~{CS}{slash}SHDN)")
+	)
+	(segment
+		(start 147.955 80.645)
+		(end 148.59 80.01)
+		(width 0.2)
+		(layer "F.Cu")
+		(net "Net-(U2-Vref)")
+	)
+	(segment
+		(start 142.24 86.995)
+		(end 145.415 83.82)
+		(width 0.2)
+		(layer "F.Cu")
+		(net "Net-(U2-Vref)")
+	)
+	(segment
+		(start 147.955 82.55)
+		(end 147.955 80.645)
+		(width 0.2)
+		(layer "F.Cu")
+		(net "Net-(U2-Vref)")
+	)
+	(segment
+		(start 137.795 86.995)
+		(end 142.24 86.995)
+		(width 0.2)
+		(layer "F.Cu")
+		(net "Net-(U2-Vref)")
+	)
+	(segment
+		(start 146.685 83.82)
+		(end 147.955 82.55)
+		(width 0.2)
+		(layer "F.Cu")
+		(net "Net-(U2-Vref)")
+	)
+	(segment
+		(start 145.415 83.82)
+		(end 146.685 83.82)
+		(width 0.2)
+		(layer "F.Cu")
+		(net "Net-(U2-Vref)")
+	)
+	(segment
+		(start 148.59 80.01)
+		(end 150.495 80.01)
+		(width 0.2)
+		(layer "F.Cu")
+		(net "Net-(U2-Vref)")
+	)
+	(segment
 		(start 130.575 77.705)
 		(end 133.35 74.93)
@@
 	)
 	(segment
-		(start 130.175 95.25)
-		(end 137.795 102.87)
-		(width 0.2)
-		(layer "B.Cu")
-		(net "Net-(J2-Pin_17)")
-	)
-	(segment
-		(start 133.35 67.31)
-		(end 130.175 70.485)
-		(width 0.2)
-		(layer "B.Cu")
-		(net "Net-(J2-Pin_17)")
-	)
-	(segment
-		(start 130.175 70.485)
-		(end 130.175 95.25)
-		(width 0.2)
-		(layer "B.Cu")
-		(net "Net-(J2-Pin_17)")
-	)
-	(segment
 		(start 135.89 76.2)
 		(end 132.715 79.375)
@@
 	)
 	(segment
-		(start 133.367 36.857)
-		(end 133.394 36.83)
-		(width 0.2)
-		(layer "F.Cu")
-		(net "unconnected-(J2-Pin_5-Pad5)")
-	)
-	(segment
 		(start 133.367 34.317)
 		(end 133.361911 34.311911)
@@
 		(net "unconnected-(J2-Pin_4-Pad4)")
 	)
+	(segment
+		(start 133.367 36.857)
+		(end 133.394 36.83)
+		(width 0.2)
+		(layer "F.Cu")
+		(net "unconnected-(J2-Pin_5-Pad5)")
+	)
 	(zone

Commit message: C12666MA PCB V2.0
Parts:
- removed A1: RaspberryPi_Pico, Module:RaspberryPi_Pico_Common_Unspecified
- removed U3: OPA340P, Package_DIP:DIP-8_W7.62mm
- removed U7: MCP1541-I/TO, Library JII FP:MCP1541_I_TO
- added C2: 0.1 μF, Capacitor_SMD:C_0805_2012Metric_Pad1.18x1.45mm_HandSolder, F.Cu at (133.9, 88.4)
- added C3: 0.1 μF, Capacitor_SMD:C_0805_2012Metric_Pad1.18x1.45mm_HandSolder, F.Cu at (147.6, 69.8)
- added C4: 0,1μF, Capacitor_SMD:C_0805_2012Metric_Pad1.18x1.45mm_HandSolder, F.Cu at (147.6, 32.0)
- added C5: 0.1 μF, Capacitor_SMD:C_0805_2012Metric_Pad1.18x1.45mm_HandSolder, F.Cu at (147.6, 76.7)
- added C6: 0.1 μF, Capacitor_SMD:C_0805_2012Metric_Pad1.18x1.45mm_HandSolder, F.Cu at (147.6, 27.7)
- added C7: 1μF, Capacitor_SMD:C_0805_2012Metric_Pad1.18x1.45mm_HandSolder, F.Cu at (144.3, 82.5)
- added REF**: PinHeader_1x01_P1.00mm_Vertical, Connector_PinHeader_1.00mm:PinHeader_1x01_P1.00mm_Vertical, F.Cu at (137.7, 82.5)
- added U1: MCP1541-I_TO, Library JII FP:MCP1541-I-TO, F.Cu at (148.4, 80.3)
- C1: footprint Capacitor_THT:C_Rect_L4.6mm_W2.0mm_P2.50mm_MKS02_FKP02 -> Capacitor_SMD:C_0805_2012Metric_Pad1.18x1.45mm_HandSolder
- R1: value 50Ω -> 5KΩ; footprint Resistor_THT:R_Axial_DIN0204_L3.6mm_D1.6mm_P7.62mm_Horizontal -> Resistor_SMD:R_0805_2012Metric_Pad1.20x1.40mm_HandSolder
- moved U6 50.6 mm to (144.5, 65.0)
- moved C1 42.0 mm to (147.3, 50.8), turned to 90 degrees
- moved U4 34.5 mm to (138.2, 87.6)
- moved U2 16.5 mm to (136.9, 70.6)
- moved R1 2.44 mm to (133.9, 81.5), turned to 90 degrees
- moved U5 1.61 mm to (144.5, 43.7)
Connections:
- C1 pad 1: Net-(U2-IN+) -> GND
- C1 pad 2: GND -> +5V
- R1 pad 1: Net-(U3--) -> Net-(U4-Video)
- U4 pad 2: Net-(U3-+) -> Net-(U4-Video)
Routing:
- net +5V: track 0.00 -> 108.5 mm, vias 0 -> 4
- net Net-(U4-CLK): track 38.0 -> 72.8 mm
- net Net-(U4-ST): track 29.7 -> 62.9 mm
- net Net-(U4-GAIN): track 23.2 -> 55.5 mm
- net Net-(J2-Pin_19): track 41.5 -> 13.9 mm
- net Net-(U3-+): track 25.8 -> 0.00 mm
- net Net-(J2-Pin_17): track 40.0 -> 16.5 mm
- net Net-(U3--): track 15.1 -> 0.00 mm
- net Net-(J1-Pin_5): track 30.4 -> 16.4 mm
- net Net-(U4-Video): track 0.00 -> 13.7 mm
- net Net-(J2-Pin_20): track 28.7 -> 17.7 mm
- net Net-(J1-Pin_4): track 25.8 -> 15.6 mm
- net Net-(U2-~{CS}/SHDN): track 22.3 -> 19.0 mm, vias 0 -> 2
- net Net-(U1-VOUT): track 16.7 -> 18.1 mm
- net Net-(U2-CLK): track 22.6 -> 21.4 mm
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- added copper zone on F.Cu, net GND
- removed copper zone on F.Cu, net +5V
Other:
- board size 24.8 x 96.5 mm -> 24.8 x 86.4 mm
- board text removed: "Video"
