File: kicad/Raspberry pico board.kicad_sch (KiCad schematic)
At the start: 11 parts, among them J1 Conn_01x20_Socket, J2 Conn_01x20_Socket, U2 MCP3301, U3 OPA340P, U4 C12666MA, U5 SN74AHCT125N, U6 SN74AHCT125N, U7 MCP1541-I/TO

Commit message: Schematic V2.0 finally made it work :)
Parts:
- removed C1: 0.1 μF, Capacitor_SMD:C_0805_2012Metric_Pad1.18x1.45mm_HandSolder, symbol Device:C_Small
- removed U3: OPA340P, Package_DIP:DIP-8_W7.62mm, symbol Amplifier_Operational:OPA340P
- added C1, C2, C3, C5, C6: 0.1 μF, symbol Device:C
- added C4: 0,1μF, symbol Device:C
- added C7: 1μF, symbol Device:C
- R1: value 50Ω -> 5KΩ
Connections:
- net +5V: now also C1.2, C2.2, C3.2, C4.1, C5.2, C6.2
- net GND: now also C1.1, C2.1, C3.1, C4.2, C5.1, C6.1, C7.2
- net at U2.1 (Vref), U7.2 (VOUT): now also C7.1
- net at R1.1: now also U4.2 (Video)
Other:
- title: (none) -> C12666Board v2
- moved on the sheet: R1, U2, U4, U5, U7

Commit message: C12666MA PCB V2.0
Parts:
- removed U7: MCP1541-I/TO, Library JII FP:MCP1541_I_TO, symbol Library JII:MCP1541-I_TO
- added U1: MCP1541-I_TO, MCP1541-I_TO:TO127P254X495-3, symbol Library JII:MCP1541-I_TO
Connections:
- net +5V: now also U1.3 (VIN)
- net GND: now also U1.1 (VSS)
- net at C7.1, U2.1 (Vref): now also U1.2 (VOUT)
Other:
- company: (none) -> Jan Ingenhousz Institute
- title: C12666Board v2 -> C12666MA Board v2
- moved on the sheet: C3

Commit message: Gui Change
Parts:
- added C8: 0,1μF, symbol Device:C
Changed lines of the file:
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@@
+	(symbol
+		(lib_id "Device:C")
+		(at 76.2 171.45 0)
+		(unit 1)
+		(body_style 1)
+		(exclude_from_sim no)
+		(in_bom yes)
+		(on_board yes)
+		(in_pos_files yes)
+		(dnp no)
+		(property "Reference" "C8"
+			(at 77.978 175.768 90)
+			(show_name no)
+			(do_not_autoplace no)
+			(effects
+				(font
+					(size 1.27 1.27)
+				)
+				(justify left)
+			)
+		)
+		(property "Value" "0,1μF"
+			(at 80.264 173.228 90)
+			(show_name no)
+			(do_not_autoplace no)
+			(effects
+				(font
+					(size 1.27 1.27)
+				)
+				(justify left)
+			)
+		)
+		(property "Footprint" ""
+			(at 77.1652 175.26 0)
+			(hide yes)
+			(show_name no)
+			(do_not_autoplace no)
+			(effects
+				(font
+					(size 1.27 1.27)
+				)
+			)
+		)
+		(property "Datasheet" ""
+			(at 76.2 171.45 0)
+			(hide yes)
+			(show_name no)
+			(do_not_autoplace no)
+			(effects
+				(font
+					(size 1.27 1.27)
+				)
+			)
+		)
+		(property "Description" "Unpolarized capacitor"
+			(at 76.2 171.45 0)
+			(hide yes)
+			(show_name no)
+			(do_not_autoplace no)
+			(effects
+				(font
+					(size 1.27 1.27)
+				)
+			)
+		)
+		(pin "1"
+		)
+		(pin "2"
+		)
+		(instances
+			(project "Raspberry pico board"
+				(path "/81531308-61af-4f59-a14f-8eee88cccc1e"
+					(reference "C8")
+					(unit 1)
+				)
+			)
+		)
+	)
 	(symbol
 		(lib_id "Device:C")
@@
 					(unit 1)
 				)
+			)
+		)
+	)
+	(symbol
+		(lib_id "power:GND")
+		(at 83.82 176.53 0)
+		(unit 1)
+		(body_style 1)
+		(exclude_from_sim no)
+		(in_bom yes)
+		(on_board yes)
+		(in_pos_files yes)
+		(dnp no)
+		(fields_autoplaced yes)
+		(property "Reference" "#PWR021"
+			(at 83.82 182.88 0)
+			(hide yes)
+			(show_name no)
+			(do_not_autoplace no)
+			(effects
+				(font
+					(size 1.27 1.27)
+				)
+			)
+		)
+		(property "Value" "GND"
+			(at 83.82 181.61 0)
+			(show_name no)
+			(do_not_autoplace no)
+			(effects
+				(font
+					(size 1.27 1.27)
+				)
+			)
+		)
+		(property "Footprint" ""
+			(at 83.82 176.53 0)
+			(hide yes)
+			(show_name no)
+			(do_not_autoplace no)
+			(effects
+				(font
+					(size 1.27 1.27)
+				)
+			)
+		)
+		(property "Datasheet" ""
+			(at 83.82 176.53 0)
+			(hide yes)
+			(show_name no)
+			(do_not_autoplace no)
+			(effects
+				(font
+					(size 1.27 1.27)
+				)
+			)
+		)
+		(property "Description" "Power symbol creates a global label with name \"GND\" , ground"
+			(at 83.82 176.53 0)
+			(hide yes)
+			(show_name no)
+			(do_not_autoplace no)
+			(effects
+				(font
+					(size 1.27 1.27)
+				)
+			)
+		)
+		(pin "1"
+		)
+		(instances
+			(project "Raspberry pico board"
+				(path "/81531308-61af-4f59-a14f-8eee88cccc1e"
+					(reference "#PWR021")
+					(unit 1)
+				)
